Commit message: feature: broken the gazebo definitions of the robot out into new file, working on getting the robot physical parameters straight. This has broken docker launch of gazebo (again\!)

File: ros_ws/src/mobile_robot_gazebo/urdf/mobile_robot_basic.urdf.xacro (robot description, xacro)
@@ -1,5 +1,5 @@
 <?xml version="1.0"?>
 <!--
-    Mobile Robot: Basic URDF and XACRO Definition
+    Mobile Robot: Mobile Robot URDF and XACRO Definition
     Iain Brookshaw
     Copyright (c), 2019. All Rights Reserved
@@ -11,21 +11,24 @@
 <robot name="mobile_robot_basic" xmlns:xacro="http://ros.org/wiki/xacro">
     <!--
-        Define some Constants
+        Define Robot Constants
+        These are for geometry only. Physics constants for the simulator
+        are in <name>.gazebo
     -->
     <!-- Chassis Constants -->
-    <xacro:property name="chassis_height"        value="0.1"     />
-    <xacro:property name="chassis_center"        value="0 0 0.3" />
-    <xacro:property name="chassis_mass"          value="1.0"     />
-    <!-- Drive Wheel Constants -->
-    <xacro:property name="wheel_base"            value="0.2"  />
-    <xacro:property name="wheel_diameter"        value="0.07" />
-    <xacro:property name="wheel_thickness"       value="0.01" />
-    <xacro:property name="wheel_mass"            value="0.01" />
-    <!-- castor wheel constants -->
-    <xacro:property name="castor_wheel_diameter" value="0.05" />
-    <xacro:property name="castor_wheel_center"   value="-0.1 0 0.025" />
-    <!--
-        Define a macro to compute the default inertial value for an object
-    -->
+    <xacro:property name="chassis_height"   value="0.05"     />
+    <xacro:property name="chassis_diameter" value="0.2"      />
+    <xacro:property name="chassis_center"   value="0 0 ${chassis_height / 2.0}" />
+    <xacro:property name="chassis_mass"     value="1.0"      />
+    <!-- Drive Wheels Constants -->
+    <xacro:property name="wheel_base"      value="${chassis_diameter}"/>
+    <xacro:property name="wheel_diameter"  value="0.05"  />
+    <xacro:property name="wheel_thickness" value="0.005" />
+    <xacro:property name="wheel_mass"      value="0.001" />
+    <xacro:property name="wheel_axel_x"    value="0.01" />
+    <!-- Castor Wheel Constants -->
+    <xacro:property name="castor_wheel_diameter" value="0.03" />
+    <xacro:property name="castor_wheel_center"   value="-${chassis_diameter/2.0} 0 ${castor_wheel_diameter/2.0}" />
+    <xacro:property name="castor_wheel_mass"     value="0.001" />
+    <!-- Define a macro to compute the default inertial value for a link -->
     <xacro:macro name="default_inertial" params="mass">
         <inertial>
@@ -34,11 +37,14 @@
         </inertial>
     </xacro:macro>
-    <!--
-        Robot Chassis Link
+    <!-- load the physics constants for the Gazebo Simulator -->
+    <xacro:include filename="$(find mobile_robot_gazebo)/urdf/mobile_robot_basic.gazebo" />
+    <!-- _______________________________________________________________________________________________________________
+         LINKS & JOINTS
     -->
+    <!-- Robot Chassis Link -->
     <link name="chassis">
         <visual>
             <geometry>
-                <cylinder radius="${wheel_base}" length="${chassis_height}"/>
+                <cylinder radius="${chassis_diameter/2.0}" length="${chassis_height}"/>
                 <origin xyz="${chassis_center}" />
             </geometry>
@@ -46,5 +52,5 @@
         <collision>
             <geometry>
-                <cylinder radius="${wheel_base}" length="${chassis_height}"/>
+                <cylinder radius="${chassis_diameter/2.0}" length="${chassis_height}"/>
                 <origin xyz="${chassis_center}" />
             </geometry>
@@ -53,7 +59,5 @@
         <!-- TODO: GAZEBO PLUGIN FOR SENSORS GOES HERE -->
     </link>
-    <!--
-        Castor Wheel Link and Joint
-    -->
+    <!-- Castor Wheel Link and Joint -->
     <link name="castor_wheel">
         <visual>
@@ -69,9 +73,10 @@
             </geometry>
         </collision>
+        <xacro:default_inertial mass="${castor_wheel_mass}"/>
     </link>
     <joint name="castor_joint" type="fixed">
         <parent link="chassis"      />
         <child  link="castor_wheel" />
-        <origin xyz="0 0 -${castor_wheel_diameter/2.0}" rpy="0 0 0"/>
+        <origin xyz="0 0 -${chassis_height}" rpy="0 0 0"/>
     </joint>
     <!--
@@ -100,15 +105,6 @@
             <parent link="chassis" />
             <child link="${prefix}_wheel"/>
-            <origin xyz="0 ${wheel_base*reflect/2.0} -${wheel_diameter/2+.05}" rpy="0 0 0"/>
+            <origin xyz="${wheel_axel_x} ${0.005*reflect + wheel_base*reflect/2.0} -${wheel_diameter/2.0}" rpy="0 0 0"/>
         </joint>
-        <!-- This block provides the simulator (Gazebo) with information on a few additional
-        physical properties. See http://gazebosim.org/tutorials/?tut=ros_urdf for more-->
-        <gazebo reference="${prefix}_wheel">
-            <mu1 value="200.0"/>
-            <mu2 value="100.0"/>
-            <kp value="10000000.0" />
-            <kd value="1.0" />
-        </gazebo>
-        <!-- TODO: WHEEL PLUGIN FOR MOTOR GOES HERE -->
     </xacro:macro>
     <!--

Commit message: feature: robot motor controllers are now in place and the robot can move...

File: ros_ws/src/mobile_robot_gazebo/urdf/mobile_robot_basic.urdf.xacro (robot description, xacro)
@@ -37,9 +37,14 @@
         </inertial>
     </xacro:macro>
-    <!-- load the physics constants for the Gazebo Simulator -->
+    <!-- load the physics constants and other elements needed for the Gazebo Simulator -->
     <xacro:include filename="$(find mobile_robot_gazebo)/urdf/mobile_robot_basic.gazebo" />
     <!-- _______________________________________________________________________________________________________________
          LINKS & JOINTS
     -->
+    <!-- Dummy Base Link
+         This is here because "KDL does not support a root link with an inertia"
+         https://answers.ros.org/question/192817/error-msg-the-root-link_base-has-an-inertia-specified-in-the-urdf-but-kdl/
+    -->
+    <link name="dummy_base_link"/>
     <!-- Robot Chassis Link -->
     <link name="chassis">
@@ -57,6 +62,9 @@
         </collision>
         <xacro:default_inertial mass="${chassis_mass}"/>
-        <!-- TODO: GAZEBO PLUGIN FOR SENSORS GOES HERE -->
     </link>
+    <joint name="dummy_base_joint" type="fixed">
+        <parent link="dummy_base_link"/>
+        <child  link="chassis"/>
+    </joint>
     <!-- Castor Wheel Link and Joint -->
     <link name="castor_wheel">
@@ -81,5 +89,5 @@
     </joint>
     <!--
-        Drive Wheel Links and Joints
+        Drive Wheel Links, Joints and Transmission
         These are defined as an XACRO macro to make them duplicates
         mirror using the 'reflect' param: 1 is one side -1 the other
@@ -107,4 +115,14 @@
             <origin xyz="${wheel_axel_x} ${0.005*reflect + wheel_base*reflect/2.0} -${wheel_diameter/2.0}" rpy="0 0 0"/>
         </joint>
+        <transmission name="${prefix}_motor_transmission">
+            <type>transmission_interface/SimpleTransmission</type>
+                <joint name="${prefix}_wheel_joint">
+                    <hardwareInterface>hardware_interface/EffortJointInterface</hardwareInterface>
+                </joint>
+                <actuator name="${prefix}_motor">
+                    <hardwareInterface>hardware_interface/EffortJointInterface</hardwareInterface>
+                    <mechanicalReduction>1</mechanicalReduction>
+                </actuator>
+        </transmission>
     </xacro:macro>
     <!--
