Commit message: IB/models: have basic xacro arch and layout complete

File: ning_ros_workspace/src/ning_urdf/urdf/math.xacro (robot description, xacro)
@@ -7,9 +7,11 @@
     Useful math utils for all geometries
 -->
- <!-- Define a macro to compute the default inertial value for a link -->
-<xacro:macro name="default_inertial" params="mass">
-    <inertial>
-        <mass value="${mass}" />
-        <inertia ixx="1.0" ixy="0.0" ixz="0.0" iyy="1.0" iyz="0.0" izz="1.0" />
-    </inertial>
-</xacro:macro>
+<robot name="ningauble" xmlns:xacro="http://ros.org/wiki/xacro">
+    <!-- Define a macro to compute the default inertial value for a link -->
+    <xacro:macro name="default_inertial" params="mass">
+        <inertial>
+            <mass value="${mass}" />
+            <inertia ixx="1.0" ixy="0.0" ixz="0.0" iyy="1.0" iyz="0.0" izz="1.0" />
+        </inertial>
+    </xacro:macro>
+</robot>

File: ning_ros_workspace/src/ning_urdf/urdf/sensor_head.xacro (robot description, xacro)
@@ -10,3 +10,9 @@
         <!-- TODO: Implement -->
     </link>
+    <joint name="neck_joint" type="continuous" >
+        <axis xyz="0 0 1" rpy="0 0 0"/>
+        <parent link="chassis" />
+        <child link="sensor_head" />
+        <origin xyz="0 0 0" rpy="0 0 0" />
+    </joint>
 </robot>

File: ning_ros_workspace/src/ning_urdf/urdf/wheel.xacro (robot description, xacro)
@@ -6,35 +6,38 @@
     MIT License
 -->
-<!-- Drive Wheels Constants -->
-<xacro:property name="wheel_diameter"  value="0.05"  />
-<xacro:property name="wheel_thickness" value="0.005" />
-<xacro:property name="wheel_mass"      value="0.001" />
-<xacro:property name="wheel_axel_x"    value="0.01" />
-<!--
-    Drive Wheel Links and Joints
-    These are defined as an XACRO macro to make them duplicates
-    mirror using the 'reflect' param: 1 is one side -1 the other
--->
-<xacro:macro name="wheel" params="prefix reflect">
-    <link name="${prefix}_wheel">
-        <visual>
-            <origin xyz="0 0 0" rpy="${pi/2} 0 0" />
-            <geometry>
-                <cylinder radius="${wheel_diameter/2.0}" length="${wheel_thickness}"/>
-            </geometry>
-        </visual>
-        <collision>
-            <origin xyz="0 0 0" rpy="${pi/2} 0 0" />
-            <geometry>
-                <cylinder radius="${wheel_diameter/2}" length="${wheel_thickness}"/>
-            </geometry>
-        </collision>
-        <xacro:default_inertial mass="${wheel_mass}"/>
-    </link>
-    <joint name="${prefix}_wheel_joint" type="continuous" >
-        <axis xyz="0 1 0" rpy="0 0 0" />
-        <parent link="chassis" />
-        <child link="${prefix}_wheel"/>
-        <origin xyz="${wheel_axel_x} ${0.005*reflect + wheel_base*reflect/2.0} -${wheel_diameter/2.0}" rpy="0 0 0"/>
-    </joint>
-</xacro:macro>
+<robot name="ningauble" xmlns:xacro="http://ros.org/wiki/xacro">
+    <!-- Drive Wheels Constants -->
+    <xacro:property name="wheel_diameter"  value="0.05"  />
+    <xacro:property name="wheel_thickness" value="0.005" />
+    <xacro:property name="wheel_mass"      value="0.001" />
+    <xacro:property name="wheel_axel_x"    value="0.01"  />
+    <xacro:property name="wheel_base"      value="0.30"  />
+    <!--
+        Drive Wheel Links and Joints
+        These are defined as an XACRO macro to make them duplicates
+        mirror using the 'reflect' param: 1 is one side -1 the other
+    -->
+    <xacro:macro name="wheel" params="prefix reflect">
+        <link name="${prefix}_wheel">
+            <visual>
+                <origin xyz="0 0 0" rpy="${pi/2} 0 0" />
+                <geometry>
+                    <cylinder radius="${wheel_diameter/2.0}" length="${wheel_thickness}"/>
+                </geometry>
+            </visual>
+            <collision>
+                <origin xyz="0 0 0" rpy="${pi/2} 0 0" />
+                <geometry>
+                    <cylinder radius="${wheel_diameter/2}" length="${wheel_thickness}"/>
+                </geometry>
+            </collision>
+            <xacro:default_inertial mass="${wheel_mass}"/>
+        </link>
+        <joint name="${prefix}_wheel_joint" type="continuous" >
+            <axis xyz="0 1 0" rpy="0 0 0" />
+            <parent link="chassis" />
+            <child link="${prefix}_wheel"/>
+            <origin xyz="${wheel_axel_x} ${0.005*reflect + wheel_base*reflect/2.0} -${wheel_diameter/2.0}" rpy="0 0 0"/>
+        </joint>
+    </xacro:macro>
+</robot>
