Commit message: IB/models: can stand up and load a model (model xacro is broken, but that's easy-ier to fix

File: ning_ros_workspace/src/ning_urdf/urdf/sensor_head.xacro (robot description, xacro)
@@ -8,5 +8,16 @@
 <robot name="ningauble" xmlns:xacro="http://ros.org/wiki/xacro">
     <link name="sensor_head">
-        <!-- TODO: Implement -->
+        <collision name="sensor_head_collision">
+            <origin xyz="0 0 0" rpy="0 0 0" />
+            <geometry>
+                <cylinder radius="0.15" length="0.2" />
+            </geometry>
+        </collision>
+        <visual name="sensor_head_visual">
+            <origin xyz="0 0 0" rpy="0 0 0" />
+            <geometry>
+                <cylinder radius="0.15" length="0.2" />
+            </geometry>
+        </visual>
     </link>
     <joint name="neck_joint" type="continuous" >

File: ning_ros_workspace/src/ning_urdf/urdf/wheel.xacro (robot description, xacro)
@@ -18,7 +18,7 @@
         mirror using the 'reflect' param: 1 is one side -1 the other
     -->
-    <xacro:macro name="wheel" params="prefix reflect">
+    <xacro:macro name="wheel" params="prefix reflect_x reflect_y">
         <link name="${prefix}_wheel">
-            <visual>
+            <visual name="${prefix}_wheel_visual">
                 <origin xyz="0 0 0" rpy="${pi/2} 0 0" />
                 <geometry>
@@ -26,5 +26,5 @@
                 </geometry>
             </visual>
-            <collision>
+            <collision name="${prefix}_wheel_collision">
                 <origin xyz="0 0 0" rpy="${pi/2} 0 0" />
                 <geometry>
@@ -38,5 +38,5 @@
             <parent link="chassis" />
             <child link="${prefix}_wheel"/>
-            <origin xyz="${wheel_axel_x} ${0.005*reflect + wheel_base*reflect/2.0} -${wheel_diameter/2.0}" rpy="0 0 0"/>
+            <origin xyz="${reflect_x*wheel_base/2.0} ${reflect_y*wheel_base/2.0} ${wheel_diameter/2.0}" rpy="0 0 0"/>
         </joint>
     </xacro:macro>

File: ning_ros_workspace/src/ning_urdf/urdf/x_drive_base.xacro (robot description, xacro)
@@ -10,7 +10,7 @@
 <robot name="ningauble" xmlns:xacro="http://ros.org/wiki/xacro">
     <xacro:include filename="$(find ning_urdf)/urdf/wheel.xacro" />
-    <xacro:wheel prefix="forward_left"  reflect="-1" />
-    <xacro:wheel prefix="forward_right" reflect="1"  />
-    <xacro:wheel prefix="back_left"  reflect="-1" />
-    <xacro:wheel prefix="back_right" reflect="1"  />
+    <xacro:wheel prefix="forward_left"  reflect_x="-1" reflect_y="1"/>
+    <xacro:wheel prefix="forward_right" reflect_x="1"  reflect_y="1"/>
+    <xacro:wheel prefix="back_left"  reflect_x="1" reflect_y="-1" />
+    <xacro:wheel prefix="back_right" reflect_x="1" reflect_y="1"  />
 </robot>
