Commit message: broken the ning xacros into sub-components

File: ning_ros_workspace/src/ning_urdf/urdf/ningauble.xacro (robot description, xacro)
@@ -5,109 +5,15 @@
     Copyright (c), 2020. All Rights Reserved
     MIT License
-    This should work with both Gazebo and RViz
-    see https://github.com/ros/urdf_sim_tutorial/blob/master/urdf/13-diffdrive.urdf.xacro
-    for a base example
+    Master Xacro file for the Ningauble robot, all major components are imported
+    to this file to assemble this modular machine
+    see: https://github.com/ros/urdf_sim_tutorial/blob/master/urdf/13-diffdrive.urdf.xacro
 -->
 <robot name="ningauble" xmlns:xacro="http://ros.org/wiki/xacro">
-    <!--
-        Define Robot Constants
-        These are for geometry only. Physics constants for the simulator
-        are in ningauble.gazebo
-    -->
-    <!-- Chassis Constants -->
-    <xacro:property name="chassis_height"   value="0.05"     />
-    <xacro:property name="chassis_diameter" value="0.2"      />
-    <xacro:property name="chassis_center"   value="0 0 ${chassis_height / 2.0}" />
-    <xacro:property name="chassis_mass"     value="1.0"      />
-    <!-- Drive Wheels Constants -->
-    <xacro:property name="wheel_base"      value="${chassis_diameter}"/>
-    <xacro:property name="wheel_diameter"  value="0.05"  />
-    <xacro:property name="wheel_thickness" value="0.005" />
-    <xacro:property name="wheel_mass"      value="0.001" />
-    <xacro:property name="wheel_axel_x"    value="0.01" />
-    <!-- Castor Wheel Constants -->
-    <xacro:property name="castor_wheel_diameter" value="0.03" />
-    <xacro:property name="castor_wheel_center"   value="-${chassis_diameter/2.0} 0 ${castor_wheel_diameter/2.0}" />
-    <xacro:property name="castor_wheel_mass"     value="0.001" />
-    <!-- Define a macro to compute the default inertial value for a link -->
-    <xacro:macro name="default_inertial" params="mass">
-        <inertial>
-            <mass value="${mass}" />
-            <inertia ixx="1.0" ixy="0.0" ixz="0.0" iyy="1.0" iyz="0.0" izz="1.0" />
-        </inertial>
-    </xacro:macro>
-    <!-- load the physics constants for the Gazebo Simulator -->
+    <!-- MUST be included first -->
+    <xacro:include filename="$(find ning_urdf)/urdf/math.xacro" />
+    <!-- actual robot components -->
+    <xacro:include filename="$(find ning_urdf)/urdf/chassis.xacro" />
+    <xacro:include filename="$(find ning_urdf)/urdf/sensor_head.xacro" />
+    <xacro:include filename="$(find ning_urdf)/urdf/x_drive_base.xacro" />
     <xacro:include filename="$(find ning_urdf)/urdf/ningauble.gazebo" />
-    <!-- _______________________________________________________________________________________________________________
-         LINKS & JOINTS
-    -->
-    <link name="chassis">
-        <visual>
-            <geometry>
-                <cylinder radius="${chassis_diameter/2.0}" length="${chassis_height}"/>
-                <origin xyz="${chassis_center}" />
-            </geometry>
-        </visual>
-        <collision>
-            <geometry>
-                <cylinder radius="${chassis_diameter/2.0}" length="${chassis_height}"/>
-                <origin xyz="${chassis_center}" />
-            </geometry>
-        </collision>
-        <xacro:default_inertial mass="${chassis_mass}"/>
-        <!-- TODO: GAZEBO PLUGIN FOR SENSORS GOES HERE -->
-    </link>
-    <link name="castor_wheel">
-        <visual>
-            <origin xyz="${castor_wheel_center}" />
-            <geometry>
-                <sphere radius="${castor_wheel_diameter/2.0}" />
-            </geometry>
-        </visual>
-        <collision>
-            <origin xyz="${castor_wheel_center}" />
-            <geometry>
-                <sphere radius="${castor_wheel_diameter/2.0}" />
-            </geometry>
-        </collision>
-        <xacro:default_inertial mass="${castor_wheel_mass}"/>
-    </link>
-    <joint name="castor_joint" type="fixed">
-        <parent link="chassis"      />
-        <child  link="castor_wheel" />
-        <origin xyz="0 0 -${chassis_height}" rpy="0 0 0"/>
-    </joint>
-    <!--
-        Drive Wheel Links and Joints
-        These are defined as an XACRO macro to make them duplicates
-        mirror using the 'reflect' param: 1 is one side -1 the other
-    -->
-    <xacro:macro name="wheel" params="prefix reflect">
-        <link name="${prefix}_wheel">
-            <visual>
-                <origin xyz="0 0 0" rpy="${pi/2} 0 0" />
-                <geometry>
-                    <cylinder radius="${wheel_diameter/2.0}" length="${wheel_thickness}"/>
-                </geometry>
-            </visual>
-            <collision>
-                <origin xyz="0 0 0" rpy="${pi/2} 0 0" />
-                <geometry>
-                    <cylinder radius="${wheel_diameter/2}" length="${wheel_thickness}"/>
-                </geometry>
-            </collision>
-            <xacro:default_inertial mass="${wheel_mass}"/>
-        </link>
-        <joint name="${prefix}_wheel_joint" type="continuous" >
-            <axis xyz="0 1 0" rpy="0 0 0" />
-            <parent link="chassis" />
-            <child link="${prefix}_wheel"/>
-            <origin xyz="${wheel_axel_x} ${0.005*reflect + wheel_base*reflect/2.0} -${wheel_diameter/2.0}" rpy="0 0 0"/>
-        </joint>
-    </xacro:macro>
-    <!--
-        Run the wheel macros to create the left and right wheels
-    -->
-    <xacro:wheel prefix="left"  reflect="-1" />
-    <xacro:wheel prefix="right" reflect="1"  />
 </robot>

Commit message: IB/ning-models: working on a ros-runner docker image to run most ros stuff... I need this to validate xacro, to then create model, to then write stuff..

File: ning_ros_workspace/src/ning_urdf/urdf/ningauble.xacro (robot description, xacro)
@@ -26,8 +26,6 @@
     <xacro:property name="wheel_mass"      value="0.001" />
     <xacro:property name="wheel_axel_x"    value="0.01" />
-    <!-- Castor Wheel Constants -->
-    <xacro:property name="castor_wheel_diameter" value="0.03" />
-    <xacro:property name="castor_wheel_center"   value="-${chassis_diameter/2.0} 0 ${castor_wheel_diameter/2.0}" />
-    <xacro:property name="castor_wheel_mass"     value="0.001" />
+    <!-- Head Constants -->
+    <xacro:property name="head_center" value="0 0 ${chassis_height / 2.0 + 1}" />
     <!-- Define a macro to compute the default inertial value for a link -->
     <xacro:macro name="default_inertial" params="mass">
@@ -45,5 +43,5 @@
         <visual>
             <geometry>
-                <cylinder radius="${chassis_diameter/2.0}" length="${chassis_height}"/>
+                <mesh filename="package://ning_urdf/urdf/meshes/dae/ningauble_torso.dae"/>
                 <origin xyz="${chassis_center}" />
             </geometry>
@@ -58,24 +56,12 @@
         <!-- TODO: GAZEBO PLUGIN FOR SENSORS GOES HERE -->
     </link>
-    <link name="castor_wheel">
+    <link name="head">
         <visual>
-            <origin xyz="${castor_wheel_center}" />
             <geometry>
-                <sphere radius="${castor_wheel_diameter/2.0}" />
+                <mesh filename="package://ning_urdf/urdf/meshes/dae/ningauble_head.dae"/>
+                <origin xyz="${head_center}" />
             </geometry>
-        </visual>
-        <collision>
-            <origin xyz="${castor_wheel_center}" />
-            <geometry>
-                <sphere radius="${castor_wheel_diameter/2.0}" />
-            </geometry>
-        </collision>
-        <xacro:default_inertial mass="${castor_wheel_mass}"/>
+        <visual>
     </link>
-    <joint name="castor_joint" type="fixed">
-        <parent link="chassis"      />
-        <child  link="castor_wheel" />
-        <origin xyz="0 0 -${chassis_height}" rpy="0 0 0"/>
-    </joint>
     <!--
         Drive Wheel Links and Joints
@@ -88,5 +74,5 @@
                 <origin xyz="0 0 0" rpy="${pi/2} 0 0" />
                 <geometry>
-                    <cylinder radius="${wheel_diameter/2.0}" length="${wheel_thickness}"/>
+                    <mesh filename="package://ning_urdf/urdf/meshes/dae/ningauble_wheel.dae"/>
                 </geometry>
             </visual>
@@ -109,5 +95,8 @@
         Run the wheel macros to create the left and right wheels
     -->
-    <xacro:wheel prefix="left"  reflect="-1" />
+    <xacro:wheel prefix="front_left"  reflect_x="-1"  reflect_y="1" />
+    <xacro:wheel prefix="front_right" reflect_x="1"   reflect_y="1" />
+    <xacro:wheel prefix="back_left"   reflect_x="-1"  reflect_y="-1" />
+    <xacro:wheel prefix="front_right" reflect_x="1"   reflect_y="-1" />
     <xacro:wheel prefix="right" reflect="1"  />
 </robot>

Commit message: sensible xacros, dockerized build script

File: ning_ros_workspace/src/ning_urdf/urdf/ningauble.xacro (robot description, xacro)
@@ -15,4 +15,5 @@
         are in ningauble.gazebo
     -->
+    <xacro:include filename="$(find ning_urdf)/urdf/math.xacro" />
     <!-- Chassis Constants -->
     <xacro:property name="chassis_height"   value="0.05"     />
@@ -28,75 +29,15 @@
     <!-- Head Constants -->
     <xacro:property name="head_center" value="0 0 ${chassis_height / 2.0 + 1}" />
-    <!-- Define a macro to compute the default inertial value for a link -->
-    <xacro:macro name="default_inertial" params="mass">
-        <inertial>
-            <mass value="${mass}" />
-            <inertia ixx="1.0" ixy="0.0" ixz="0.0" iyy="1.0" iyz="0.0" izz="1.0" />
-        </inertial>
-    </xacro:macro>
+    <xacro:property name="head_mass"   value="2.0" />
     <!-- load the physics constants for the Gazebo Simulator -->
-    <xacro:include filename="$(find ning_urdf)/urdf/ningauble.gazebo" />
-    <!-- _______________________________________________________________________________________________________________
-         LINKS & JOINTS
-    -->
-    <link name="chassis">
-        <visual>
-            <geometry>
-                <mesh filename="package://ning_urdf/urdf/meshes/dae/ningauble_torso.dae"/>
-                <origin xyz="${chassis_center}" />
-            </geometry>
-        </visual>
-        <collision>
-            <geometry>
-                <cylinder radius="${chassis_diameter/2.0}" length="${chassis_height}"/>
-                <origin xyz="${chassis_center}" />
-            </geometry>
-        </collision>
-        <xacro:default_inertial mass="${chassis_mass}"/>
-        <!-- TODO: GAZEBO PLUGIN FOR SENSORS GOES HERE -->
-    </link>
-    <link name="head">
-        <visual>
-            <geometry>
-                <mesh filename="package://ning_urdf/urdf/meshes/dae/ningauble_head.dae"/>
-                <origin xyz="${head_center}" />
-            </geometry>
-        <visual>
-    </link>
-    <!--
-        Drive Wheel Links and Joints
-        These are defined as an XACRO macro to make them duplicates
-        mirror using the 'reflect' param: 1 is one side -1 the other
-    -->
-    <xacro:macro name="wheel" params="prefix reflect">
-        <link name="${prefix}_wheel">
-            <visual>
-                <origin xyz="0 0 0" rpy="${pi/2} 0 0" />
-                <geometry>
-                    <mesh filename="package://ning_urdf/urdf/meshes/dae/ningauble_wheel.dae"/>
-                </geometry>
-            </visual>
-            <collision>
-                <origin xyz="0 0 0" rpy="${pi/2} 0 0" />
-                <geometry>
-                    <cylinder radius="${wheel_diameter/2}" length="${wheel_thickness}"/>
-                </geometry>
-            </collision>
-            <xacro:default_inertial mass="${wheel_mass}"/>
-        </link>
-        <joint name="${prefix}_wheel_joint" type="continuous" >
-            <axis xyz="0 1 0" rpy="0 0 0" />
-            <parent link="chassis" />
-            <child link="${prefix}_wheel"/>
-            <origin xyz="${wheel_axel_x} ${0.005*reflect + wheel_base*reflect/2.0} -${wheel_diameter/2.0}" rpy="0 0 0"/>
-        </joint>
-    </xacro:macro>
-    <!--
-        Run the wheel macros to create the left and right wheels
-    -->
-    <xacro:wheel prefix="front_left"  reflect_x="-1"  reflect_y="1" />
-    <xacro:wheel prefix="front_right" reflect_x="1"   reflect_y="1" />
-    <xacro:wheel prefix="back_left"   reflect_x="-1"  reflect_y="-1" />
-    <xacro:wheel prefix="front_right" reflect_x="1"   reflect_y="-1" />
-    <xacro:wheel prefix="right" reflect="1"  />
+    <!-- <xacro:include filename="$(find ning_urdf)/urdf/ningauble.gazebo" /> -->
+    <!-- Load all the Links -->
+    <xacro:include filename="$(find ning_urdf)/urdf/head.xacro" origin="${head_center}" mass="${head_mass}"/>
+    <!-- <xacro:include filename="$(find ning_urdf)/urdf/chassis/chassis.xacro"/> -->
+    <!-- <xacro:include filename="$(find ning_urdf)/urdf/legs/legs.xacro"/> -->
+    <!-- <xacro:wheel prefix="front_right" reflect_x="1"   reflect_y="1" /> -->
+    <!-- <xacro:wheel prefix="back_left"   reflect_x="-1"  reflect_y="-1" /> -->
+    <!-- <xacro:wheel prefix="front_right" reflect_x="1"   reflect_y="-1" /> -->
+    <!-- <xacro:wheel prefix="right" reflect="1"  /> -->
+    <!-- Set up all the joints -->
 </robot>
